File: sweep-half-swept/half-swept.kicad_pcb (KiCad board)
At the start: 2 copper layers, 108.9 x 86.5 mm, 22 parts, among them J2 AudioJack4dpb, SW1 SW_Push, SW10 SW_Push, SW11 SW_Push, SW12 SW_Push, SW13 SW_Push, SW14 SW_Push, SW15 SW_Push, SW16 SW_Push, SW17 SW_Push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

Commit message: adding logo to silkscreen
Parts:
- removed the G*** at (64.0, 82.0)
- added G***: LOGO, Audio_Module:Logo, F.Cu at (63.2, 81.3)
- added G***: LOGO, Audio_Module:Logo, B.Cu at (63.2, 81.3)
